File: phyphox_CO2_Monitor.kicad_pcb (KiCad board)
At the start: 2 copper layers, 80 x 38 mm, 10 parts

Commit message: horizontal design
Parts:
- removed the REF** at (51.0, 63.0)
- removed the REF** at (99.0, 91.0)
- added REF**: MountingHole_2.5mm_Pad, MountingHole:MountingHole_2.5mm_Pad, F.Cu at (18.1, 18.0)
- added REF**: MountingHole_2.5mm_Pad, MountingHole:MountingHole_2.5mm_Pad, F.Cu at (18.1, -17.6)
- added REF**: MountingHole_2.5mm_Pad, MountingHole:MountingHole_2.5mm_Pad, F.Cu at (-22.6, -17.6)
- added REF**: MountingHole_2.5mm_Pad, MountingHole:MountingHole_2.5mm_Pad, F.Cu at (-22.6, 18.0)
- R1, R2, R3, R4, R5: moved to B.Cu
- moved RGB-LED 116.2 mm to (6.02, -6.78), turned to 270 degrees
- moved R4 115.6 mm to (7.80, -7.92), turned to 270 degrees
- moved R5 115.5 mm to (14.3, -8.05), turned to 270 degrees
- moved SCD30 112.8 mm to (33.3, 0.20)
- moved R1 110.5 mm to (-6.20, 1.49)
- moved R2 110.5 mm to (-6.20, 6.49)
- moved R3 110.5 mm to (-6.20, -4.01)
- moved ESP32 110.4 mm to (0.00, 0.00)
Routing:
- net GND: track 47.5 -> 24.1 mm, vias 5 -> 4
- net SDA: track 53.6 -> 43.6 mm
- net Net-(D1-Pad4): track 10.6 -> 17.3 mm
- net SCL: track 42.3 -> 36.5 mm
- net RDY: track 59.1 -> 53.5 mm
- net Net-(D1-Pad3): track 9.04 -> 12.4 mm
- net VDD: track 74.1 -> 71.0 mm, vias 1 -> 0
- net GREEN: track 37.7 -> 40.6 mm
- net RED: track 33.2 -> 36.1 mm
- net Net-(D1-Pad1): track 9.18 -> 7.02 mm
- net BLUE: track 26.3 -> 27.7 mm
Other:
- board size 80 x 38 mm -> 73 x 42 mm

Commit message: revision 0.6
Other:
- board text added: "Rev 0.6"
- board text removed: "Rev 0.5"
Changed lines of the file:
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@@
   (gr_curve (pts (xy 40.294591 -1.90529) (xy 40.509932 -1.90529) (xy 40.537269 -1.753082) (xy 40.384671 -1.403729)) (layer B.SilkS) (width 0.01))
   (gr_curve (pts (xy 40.384671 -1.403729) (xy 40.251108 -1.097957) (xy 40.164536 -1.00529) (xy 40.012435 -1.00529)) (layer B.SilkS) (width 0.01))
-  (gr_text "Rev 0.5" (at 9.1948 17.9832) (layer F.SilkS)
-    (effects (font (size 1.5 1.5) (thickness 0.3)))
+  (gr_text "Rev 0.6" (at 9.1948 17.9832) (layer B.SilkS)
+    (effects (font (size 1.5 1.5) (thickness 0.3)) (justify mirror))
   )
   (gr_curve (pts (xy 38.047198 -2.09279) (xy 38.005995 -2.358542) (xy 37.958023 -2.702731) (xy 37.900233 -3.14724)) (layer B.SilkS) (width 0.01))

Commit message: Update to Rev 0.7
Parts:
- removed ESP32: ESP32-DEVKITC-32D, phyphox_CO2_Monitor:ESP32-DevKitC-32D
- removed RGB-LED: LED_BARG, phyphox_CO2_Monitor:WP154A4SEJ3VBDZGWCA
- removed SCD30: SCD30, phyphox_CO2_Monitor:SCD30
- added D1: LED_BARG, phyphox_CO2_Monitor:WP154A4SEJ3VBDZGWCA, B.Cu at (139.7, 78.1)
- added J1: Conn_01x19_Female, Connector_PinSocket_2.54mm:PinSocket_1x19_P2.54mm_Vertical, F.Cu at (160.8, 40.3)
- added J2: Conn_01x19_Female, Connector_PinSocket_2.54mm:PinSocket_1x19_P2.54mm_Vertical, F.Cu at (161.0, 109.9)
- added REF**: MountingHole_2.2mm_M2_DIN965_Pad, MountingHole:MountingHole_2.2mm_M2_DIN965_Pad, F.Cu at (180.7, 94.6)
- added REF**: MountingHole_2.2mm_M2_DIN965_Pad, MountingHole:MountingHole_2.2mm_M2_DIN965_Pad, F.Cu at (164.6, 62.6)
- added U1: ESP32-DEVKITC-32D, phyphox_CO2_Monitor:ESP32-DevKitC-32D, F.Cu at (141.3, 78.7)
- added U2: SCD30, phyphox_CO2_Monitor:SCD30, B.Cu at (174.5, 78.5)
- moved R3 170.0 mm to (138.0, 86.1), turned to 90 degrees
- moved R4 162.7 mm to (150.3, 70.6)
- moved R1 162.7 mm to (132.8, 86.1), turned to 90 degrees
- moved R5 161.7 mm to (155.5, 70.6)
- moved REF** 161.7 mm to (159.3, 96.7)
- moved REF** 161.7 mm to (159.3, 61.1)
- moved REF** 161.7 mm to (118.7, 61.1)
- moved REF** 161.7 mm to (118.7, 96.7)
- moved R2 156.0 mm to (127.8, 86.2), turned to 90 degrees
Routing:
- net GREEN: track 40.6 -> 14.4 mm
- net RED: track 36.1 -> 12.0 mm
- net GND: track 24.1 -> 0.00 mm, vias 4 -> 2
- net BLUE: track 27.7 -> 9.38 mm
- net VDD: track 71.0 -> 84.3 mm
- net Net-(D1-Pad1): track 7.02 -> 14.7 mm
- net Net-(D1-Pad3): track 12.4 -> 17.4 mm
- net Net-(D1-Pad4): track 17.3 -> 21.1 mm
- net RDY: track 53.5 -> 55.4 mm
- net SDA: track 43.6 -> 44.2 mm
- net SCL: track 36.5 -> 35.9 mm
Other:
- board size 73 x 42 mm -> 73.1 x 42 mm
- net class Default: trace_width 0.25 -> 0.4
- rule pad_to_mask_clearance: 0.051 -> 0
- board text added: "Rev 0.7"
- board text removed: "Rev 0.6"
