File: phyphox_CO2_Monitor.sch (KiCad schematic (older format))
At the start: 8 parts, among them U1 ESP32-DEVKITC-32D, U2 SCD30

Commit message: Update to Rev 0.7
Parts:
- added J1, J2: Conn_01x19_Female, Connector_PinSocket_2.54mm:PinSocket_1x19_P2.54mm_Vertical, symbol Connector:Conn_01x19_Female
- added J3: Conn_01x07_Male, Connector_PinHeader_2.54mm:PinHeader_1x07_P2.54mm_Vertical, symbol Connector:Conn_01x07_Male
Connections:
- wire segments 0 -> 85
Other:
- moved on the sheet: U2
